File: VFD display.kicad_pcb (KiCad board)
At the start: 2 copper layers, 100 x 62 mm, 45 parts, among them IC1 4094D, IC2 4094D, J1 SPI, J2 UART, J3 Conn_01x07_Female, Q4 2N7000, Q5 2N7000, Q6 2N7000, SW1 SW_Push, SW2 SW_Push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

Commit message: V2 Schematic updates added indication LEDs for 12V and 5V, fixed the display symbol so C is connected to pin 17, added values to the capacitors on the ADC lines, removed voltage from AREF.
Routing:
- net GND: vias 124 -> 123
- net /CLEAN 5V: vias 0 -> 1
Changed lines of the file:
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@@
   (net 60 "Net-(R19-Pad2)")
   (net 61 "Net-(R20-Pad2)")
+  (net 62 "/CLEAN 5V")
   (footprint "Capacitor_THT:C_Disc_D4.7mm_W2.5mm_P5.00mm" (layer "F.Cu")
     (at 102.8 114.57 -90)
@@
   (via (at 172 115) (size 0.8) (drill 0.4) (layers "F.Cu" "B.Cu") (net 2))
   (via (at 120.455 91.945) (size 0.8) (drill 0.4) (layers "F.Cu" "B.Cu") (free) (net 2))
-  (via (at 94.5 100) (size 0.8) (drill 0.4) (layers "F.Cu" "B.Cu") (net 2))
   (via (at 109.705 84.945) (size 0.8) (drill 0.4) (layers "F.Cu" "B.Cu") (free) (net 2))
   (via (at 158.205 83.445) (size 0.8) (drill 0.4) (layers "F.Cu" "B.Cu") (free) (net 2))
@@
   (segment (start 148.17452 122.31952) (end 181.15048 122.31952) (width 0.25) (layer "B.Cu") (net 61))
   (segment (start 182.35 121.12) (end 182.35 114.62) (width 0.25) (layer "B.Cu") (net 61))
+  (via (at 94.5 100) (size 0.8) (drill 0.4) (layers "F.Cu" "B.Cu") (net 62))
   (zone (net 2) (net_name "GND") (layers F&B.Cu) (hatch edge 0.508)
     (connect_pads (clearance 0.2))
